File: PCB/I2C Relay - Copy/relay/relay.kicad_sch (KiCad schematic)
At the start: 24 parts, among them J1 Conn_01x10_Female, J2 Conn_01x02_Female, K1 CPC1726Y, K2 CPC1726Y, K3 CPC1726Y, K4 CPC1726Y, K5 CPC1726Y, K6 CPC1726Y, K7 CPC1726Y, U1 LM317L_SOT-89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

Commit message: First Version of Optical Density source finished, swithced to a pin out connection for multispectrum LED.
Parts:
- removed LED1: LZ7-04M2PD-0000, LZ7:LZ7-04M2PD-0000, symbol 2022-02-20_03-57-01:LZ7-04M2PD-0000
- added J3: Conn_01x14_Female, Connector_PinSocket_2.54mm:PinSocket_1x14_P2.54mm_Horizontal, symbol Connector:Conn_01x14_Female
Connections:
- net A_S: now also J3.7 (Pin_7)
- net B_S: now also J3.5 (Pin_5)
- net C_S: now also J3.9 (Pin_9)
- net GND: now also J3.10 (Pin_10), J3.12 (Pin_12), J3.14 (Pin_14), J3.2 (Pin_2), J3.4 (Pin_4), J3.6 (Pin_6), J3.8 (Pin_8)
- net G_S: now also J3.3 (Pin_3)
- net L_S: now also J3.11 (Pin_11), J3.13 (Pin_13)
- net R_S: now also J3.1 (Pin_1)
- no-connect marks 17 -> 6
Other:
- note added: "Connector_PinSocket_2.54mm:PinSocket_1x10_P2.54mm_Horizontal"
- note added: "Laser Source Breakout"
- note added: "Multi-Spectrum Breakout"
- note removed: "Multi-Spectrum LED"
